Commit message: For resubmission

File: my_robot/urdf/my_robot.xacro (robot description, xacro)
@@ -10,5 +10,5 @@
     <pose>0 0 0.1 0 0 0</pose>
     <inertial>
-      <mass value="15.0"/>
+      <mass value="30.0"/>
       <origin xyz="0.0 0 0" rpy=" 0 0 0"/>
       <inertia
@@ -39,5 +39,5 @@
       <origin xyz="-0.1 0 -0.075" rpy=" 0 0 0"/>
       <geometry>
-        <sphere radius="0.075"/>
+        <sphere radius="0.073"/>
       </geometry>
     </collision>
@@ -51,5 +51,5 @@
       <origin xyz="0.1 0 -0.075" rpy=" 0 0 0"/>
       <geometry>
-        <sphere radius="0.075"/>
+        <sphere radius="0.073"/>
       </geometry>
     </collision>
@@ -61,4 +61,7 @@
     </visual>
   </link>
+  <gazebo reference="chassis">
+    <material>Gazebo/Green</material>
+  </gazebo>
   <joint type="continuous" name="mid_right_wheel_hinge">
     <origin xyz="0 -0.2 0" rpy="0 0 0"/>
@@ -72,5 +75,5 @@
     <pose>0 0 0.1 0 0 0</pose>
     <inertial>
-      <mass value="5.0"/>
+      <mass value="10.0"/>
       <origin xyz="0 0 0" rpy=" 0 1.5707 1.5707"/>
       <inertia
@@ -97,6 +100,9 @@
         <color rgba="0.0 0.0 0.0 1.0"/>
       </material>
-   </visual>
-  </link>
+    </visual>
+  </link>
+  <gazebo reference="mid_right_wheel">
+    <material>Gazebo/Black</material>
+  </gazebo>
   <joint type="continuous" name="mid_left_wheel_hinge">
     <origin xyz="0 0.2 0" rpy="0 0 0"/>
@@ -110,5 +116,5 @@
     <pose>0 0 0.1 0 0 0</pose>
     <inertial>
-      <mass value="5.0"/>
+      <mass value="10.0"/>
       <origin xyz="0 0 0" rpy=" 0 1.5707 1.5707"/>
       <inertia
@@ -137,4 +143,7 @@
     </visual>
   </link>
+  <gazebo reference="mid_left_wheel">
+    <material>Gazebo/Black</material>
+  </gazebo>
   <joint type="fixed" name="camera_joint">
     <origin xyz="0.2 0 0" rpy="0 0 0"/>
@@ -160,4 +169,7 @@
         <box size=".05 .05 .05"/>
       </geometry>
+      <material name="red">
+        <color rgba="1.0 0.0 0.0 1.0"/>
+      </material>
     </collision>
     <visual name='camera_visual'>
@@ -166,6 +178,12 @@
         <box size=".05 .05 .05"/>
       </geometry>
-    </visual>
-  </link>
+      <material name="red">
+        <color rgba="1.0 0.0 0.0 1.0"/>
+      </material>
+    </visual>
+  </link>
+  <gazebo reference="camera">
+    <material>Gazebo/Red</material>
+  </gazebo>
   <joint type="fixed" name="hokuyo_joint">
     <origin xyz="0.15 0 0.1" rpy="0 0 0"/>
